File: Motor Driver Board/Buck Conv/EVolocity Buck Conv.kicad_sch (KiCad schematic)
At the start: 52 parts, among them J1 Screw_Terminal_01x02, J2 XT30, J3 Screw_Terminal_01x02, J4 Conn_01x04, U1 NRF24L01_Breakout, U2 LM2576HVT-5, U4 L298N

Commit message: updates maybe
Parts:
- removed A2: Arduino_Nano_v3.x, Module:Arduino_Nano, symbol MCU_Module:Arduino_Nano_v3.x
- removed C13, C2, C4: 100nF, Capacitor_THT:C_Rect_L7.0mm_W2.5mm_P5.00mm, symbol Device:C
- removed C3: 10uF, Capacitor_THT:CP_Radial_D5.0mm_P2.50mm, symbol Device:C_Polarized
- removed C9: 100m, Capacitor_THT:CP_Radial_D14.0mm_P5.00mm, symbol Device:C_Polarized
- removed D12, D13, D15, D16, D17, D18, D19, D20, D21: 1N5819, Diode_THT:D_DO-41_SOD81_P7.62mm_Horizontal, symbol Device:D
- removed D14: 1N5822, Diode_THT:D_DO-41_SOD81_P7.62mm_Horizontal, symbol Device:D
- removed D2: 1N5359B, Diode_THT:D_DO-41_SOD81_P7.62mm_Horizontal, symbol Device:D_Zener
- removed D3: Green, LED_THT:LED_D3.0mm_FlatTop, symbol Device:LED
- removed D4: Red, LED_THT:LED_D3.0mm_FlatTop, symbol Device:LED
- removed D5: 1.5KE39CA (TVS), Diode_THT:D_DO-201_P12.70mm_Horizontal, symbol Diode:SZESD9B5.0ST5G
- removed F2: 1A, Resistor_THT:R_Axial_DIN0204_L3.6mm_D1.6mm_P5.08mm_Horizontal, symbol Device:Fuse
- removed J1: Screw_Terminal_01x02, TerminalBlock:TerminalBlock_MaiXu_MX126-5.0-02P_1x02_P5.00mm, symbol Connector:Screw_Terminal_01x02
- removed J2: XT30, Connector_AMASS:AMASS_XT30U-F_1x02_P5.0mm_Vertical, symbol Connector:Conn_01x02_Socket
- removed J4: Conn_01x04, Connector_PinHeader_2.54mm:PinHeader_1x04_P2.54mm_Vertical, symbol Connector_Generic:Conn_01x04
- removed R16, R17: 1k, Resistor_THT:R_Axial_DIN0207_L6.3mm_D2.5mm_P10.16mm_Horizontal, symbol Device:R
- removed R18: R_snub, Resistor_THT:R_Axial_DIN0411_L9.9mm_D3.6mm_P12.70mm_Horizontal, symbol Device:R
- removed R19: 33R, Resistor_THT:R_Axial_DIN0207_L6.3mm_D2.5mm_P10.16mm_Horizontal, symbol Device:R
- added A1: Arduino Nano, Module:Arduino_Nano, symbol MCU_Module:Arduino_Nano_v3.x
- added C10, C11, C12, C3, C8, C9: 100nF, Capacitor_THT:C_Rect_L7.0mm_W2.5mm_P5.00mm, symbol Device:C
- added C2: 470uF, Capacitor_THT:CP_Radial_D12.5mm_P5.00mm, symbol Device:C_Polarized
- added C4: 1000uF, Capacitor_THT:CP_Radial_D14.0mm_P5.00mm, symbol Device:C_Polarized
- added D1: Green, LED_THT:LED_D3.0mm_FlatTop, symbol Device:LED
- added D10, D11, D3, D4, D5, D6, D7, D8, D9: 1N5822, Diode_THT:D_DO-201AD_P15.24mm_Horizontal, symbol Device:D
- added D2: 1.5KE39CA (TVS), Diode_THT:D_DO-201_P12.70mm_Horizontal, symbol Diode:SZESD9B5.0ST5G
- added F1: 5A, Resistor_THT:R_Axial_DIN0204_L3.6mm_D1.6mm_P5.08mm_Horizontal, symbol Device:Fuse
- added J1: XT30, Connector_AMASS:AMASS_XT30U-F_1x02_P5.0mm_Vertical, symbol Connector_Generic:Conn_01x02
- added J2: Screw_Terminal_01x02, TerminalBlock:TerminalBlock_MaiXu_MX126-5.0-02P_1x02_P5.00mm, symbol Connector:Screw_Terminal_01x02
- added R14, R8: 10k, Resistor_THT:R_Axial_DIN0207_L6.3mm_D2.5mm_P10.16mm_Horizontal, symbol Device:R
- added R9: 1k, Resistor_THT:R_Axial_DIN0207_L6.3mm_D2.5mm_P10.16mm_Horizontal, symbol Device:R
- added U3: LD1117V33, Package_TO_SOT_THT:TO-220-3_Vertical, symbol Regulator_Linear:LD1117V33
- C1: value 10uF -> 100nF; footprint Capacitor_THT:CP_Radial_D5.0mm_P2.50mm -> Capacitor_THT:C_Rect_L7.0mm_W2.5mm_P5.00mm; LCSC Part No. C216300 -> C1620866; MPN (none) -> SR205C104KAR; Manufacturer (none) -> Kyocera AVX; Voltage 63V -> 50V
- C5, C6: value C_Snub -> 100nF; MPN (none) -> SR205C104KAR; Manufacturer (none) -> Kyocera AVX; Voltage (none) -> 50V
- C7: value 100nF -> 10uF; MPN (none) -> SR205C104KAR; Manufacturer (none) -> Kyocera AVX; Voltage (none) -> 50V
- H1, H2, H3, H4: now left out of the parts list
- J3: LCSC Part No. (none) -> C3819953; MPN (none) -> 1935161; Manufacturer (none) -> Phoenix Contact
- R1, R2, R3, R4, R5: value 100 -> 100R; MPN (none) -> MF0207FRE52-100R; Manufacturer (none) -> YAGEO
- R10: value 100 -> 100k; LCSC Part No. C3508583 -> C513592; MPN (none) -> MF0207FTE52-100K; Manufacturer (none) -> YAGEO
- R11: value R_snub -> 10k; footprint Resistor_THT:R_Axial_DIN0411_L9.9mm_D3.6mm_P12.70mm_Horizontal -> Resistor_THT:R_Axial_DIN0207_L6.3mm_D2.5mm_P10.16mm_Horizontal; LCSC Part No. C385291 -> C513672; MPN (none) -> MF0207FTE52-10K; Manufacturer (none) -> YAGEO
- R12, R13: value 100 -> 1k; footprint Resistor_THT:R_Axial_DIN0207_L6.3mm_D2.5mm_P10.16mm_Horizontal -> Resistor_THT:R_Axial_DIN0411_L9.9mm_D3.6mm_P12.70mm_Horizontal; LCSC Part No. C3508583 -> C385291; MPN (none) -> RN1WS1KΩFT/BA1; Manufacturer (none) -> TyoHM
- R6: value 100k -> 100R; LCSC Part No. C513592 -> C3508583; MPN (none) -> MF0207FRE52-100R; Manufacturer (none) -> YAGEO
- R7: MPN (none) -> MF0207FTE52-10K; Manufacturer (none) -> YAGEO
Connections:
- net +3V3: now also C3.1, R14.1, U3.2 (VO)
- net +5V: now also C5.1, C6.1, L1.2, U2.4 (FB), A1.27 (+5V), C10.1, C11.1, C4.1, R9.1, U3.3 (VI); no longer C1.1, R6.1, U2.1 (VIN), U2.5 (~{ON}/OFF), U4.4 (Vs)
- net EnA: now also R7.1, A1.12 (D9)
- net EnB: now also A1.13 (D10), R8.1
- net GND: now also C5.2, C6.2, R11.2, U2.5 (~{ON}/OFF), A1.29 (GND), A1.4 (GND), C10.2, C11.2, C12.2, C2.2, C3.2, C4.2, D1.1 (K), D10.2 (A), D11.2 (A), D2.2 (A2), D3.2 (A), D6.2 (A), D7.2 (A), J1.1 (Pin_1), R8.2, U3.1 (GND)
- net IN1: now also A1.7 (D4)
- net IN2: now also A1.6 (D3)
- net IN3: now also A1.8 (D5)
- net IN4: now also A1.9 (D6)
- net Radio_CE: now also R5.2; no longer R1.2
- net Radio_CS: now also R4.2, R14.2; no longer R2.2
- net Radio_MISO: now also R2.2; no longer R4.2
- net Radio_SCK: now also R1.2; no longer R5.2
- net V_Panel_Analog: now also R10.2, R11.1, A1.25 (A6), C12.1; no longer R6.2, R7.1
- net at U4.3 (OUT2): now also J3.2 (Pin_2), R12.2, D5.2 (A), D7.1 (K); no longer R11.2
- net Radio_IRQ: now reaches U1.8 (IRQ)
- net Radio_IRQ: now also R6.2
- net at L1.1, U2.2 (OUT): now also D3.1 (K); no longer U2.4 (FB)
- net at R1.1: now also A1.16 (D13)
- net at U4.14 (OUT4): now also R13.2, D11.1 (K), D9.2 (A), J2.2 (Pin_2); no longer J3.2 (Pin_2)
- net at U4.2 (OUT1): now also J3.1 (Pin_1), C9.1, D4.2 (A), D6.1 (K); no longer C5.1
- net at R4.1: now also A1.11 (D8)
- net at R2.1: now also A1.15 (D12)
- net at R3.1: now also A1.14 (D11)
- net at R5.1: now also A1.10 (D7)
- net A0 renamed PowerInput+
- net PowerInput+: now also C1.1, U2.1 (VIN), U4.4 (Vs), C2.1, D2.1 (A1), D4.1 (K), D5.1 (K), D8.1 (K), D9.1 (K), F1.2
- net A1: no longer names the net of R12.1
- net A1: now also C9.2
- net A2: no longer names the net of R13.1
- net A2: now also C8.2
- new net: C8.1, D10.1 (K), D8.2 (A), J2.1 (Pin_1), U4.13 (OUT3)
- new net: F1.1, J1.2 (Pin_2)
- new net: D1.2 (A), R9.2
- new net: A1.5 (D2), R6.1
- no-connect marks 11 -> 14
Other:
- note added: "Power Selection"
- note removed: "Extra Connector"
- note removed: "Power Backup"
- note removed: "for fun additions students want to add"
