File: Motor Driver Board/Buck Conv/EVolocity Buck Conv.kicad_sch (KiCad schematic)
At the start: 52 parts, among them J1 Screw_Terminal_01x02, J2 XT30, J3 Screw_Terminal_01x02, J4 Conn_01x04, U1 NRF24L01_Breakout, U2 LM2576HVT-5, U4 L298N

Commit message: updates after catchup
Parts:
- removed A2: Arduino_Nano_v3.x, Module:Arduino_Nano, symbol MCU_Module:Arduino_Nano_v3.x
- removed C13, C2, C4, C7: 100nF, Capacitor_THT:C_Rect_L7.0mm_W2.5mm_P5.00mm, symbol Device:C
- removed C3: 10uF, Capacitor_THT:CP_Radial_D5.0mm_P2.50mm, symbol Device:C_Polarized
- removed C5, C6: C_Snub, Capacitor_THT:C_Rect_L7.0mm_W2.5mm_P5.00mm, symbol Device:C
- removed C9: 100m, Capacitor_THT:CP_Radial_D14.0mm_P5.00mm, symbol Device:C_Polarized
- removed D12, D13, D15, D16, D17, D18, D19, D20, D21: 1N5819, Diode_THT:D_DO-41_SOD81_P7.62mm_Horizontal, symbol Device:D
- removed D14: 1N5822, Diode_THT:D_DO-41_SOD81_P7.62mm_Horizontal, symbol Device:D
- removed D2: 1N5359B, Diode_THT:D_DO-41_SOD81_P7.62mm_Horizontal, symbol Device:D_Zener
- removed D4: Red, LED_THT:LED_D3.0mm_FlatTop, symbol Device:LED
- removed D5: 1.5KE39CA (TVS), Diode_THT:D_DO-201_P12.70mm_Horizontal, symbol Diode:SZESD9B5.0ST5G
- removed F2: 1A, Resistor_THT:R_Axial_DIN0204_L3.6mm_D1.6mm_P5.08mm_Horizontal, symbol Device:Fuse
- removed J1: Screw_Terminal_01x02, TerminalBlock:TerminalBlock_MaiXu_MX126-5.0-02P_1x02_P5.00mm, symbol Connector:Screw_Terminal_01x02
- removed J2: XT30, Connector_AMASS:AMASS_XT30U-F_1x02_P5.0mm_Vertical, symbol Connector:Conn_01x02_Socket
- removed J4: Conn_01x04, Connector_PinHeader_2.54mm:PinHeader_1x04_P2.54mm_Vertical, symbol Connector_Generic:Conn_01x04
- removed L1: 100uH, Library1:IND_BOURNS_RLB1314, symbol Device:L
- removed U2: LM2576HVT-5, Package_TO_SOT_THT:TO-220-5_Vertical, symbol Regulator_Switching:LM2576HVT-5
- added A1: Arduino Nano, Module:Arduino_Nano, symbol MCU_Module:Arduino_Nano_v3.x
- added C10, C11, C12, C3, C8, C9: 100nF, Capacitor_THT:C_Rect_L7.0mm_W2.5mm_P5.00mm, symbol Device:C
- added C2: 470uF, Capacitor_THT:CP_Radial_D12.5mm_P5.00mm, symbol Device:C_Polarized
- added C4: 100nF, Capacitor_THT:C_Rect_L7.0mm_W2.5mm_P5.00mm, symbol Device:C_Polarized
- added D1: Green, LED_THT:LED_D3.0mm_FlatTop, symbol Device:LED
- added D10, D11, D4, D5, D6, D7, D8, D9: 1N5822, Diode_THT:D_DO-201AD_P15.24mm_Horizontal, symbol Device:D
- added D2: 1.5KE39CA (TVS), Diode_THT:D_DO-201_P12.70mm_Horizontal, symbol Diode:SZESD9B5.0ST5G
- added F1: 5A, Resistor_THT:R_Axial_DIN0204_L3.6mm_D1.6mm_P5.08mm_Horizontal, symbol Device:Fuse
- added J1: XT30, Connector_AMASS:AMASS_XT30U-F_1x02_P5.0mm_Vertical, symbol Connector_Generic:Conn_01x02
- added J2: Screw_Terminal_01x02, TerminalBlock:TerminalBlock_MaiXu_MX126-5.0-02P_1x02_P5.00mm, symbol Connector:Screw_Terminal_01x02
- added J4: Conn_01x05, Connector_PinHeader_2.54mm:PinHeader_1x05_P2.54mm_Vertical, symbol Connector_Generic:Conn_01x05
- added R14, R9: 1k, Resistor_THT:R_Axial_DIN0207_L6.3mm_D2.5mm_P10.16mm_Horizontal, symbol Device:R
- added R15, R8: 100R, Resistor_THT:R_Axial_DIN0207_L6.3mm_D2.5mm_P10.16mm_Horizontal, symbol Device:R
- C1: value 10uF -> 100nF; footprint Capacitor_THT:CP_Radial_D5.0mm_P2.50mm -> Capacitor_THT:C_Rect_L7.0mm_W2.5mm_P5.00mm; LCSC Part No. C216300 -> C1620866; MPN (none) -> SR205C104KAR; Manufacturer (none) -> Kyocera AVX; Voltage 63V -> 50V
- D3: LCSC Part No. C3001643 -> C3001646; MPN (none) -> TLHG4400; Manufacturer (none) -> VISHAY
- H1, H2, H3, H4: now left out of the parts list
- J3: LCSC Part No. (none) -> C3819953; MPN (none) -> 1935161; Manufacturer (none) -> Phoenix Contact
- R1, R2, R3, R4, R5: value 100 -> 100R; MPN (none) -> MF0207FRE52-100R; Manufacturer (none) -> YAGEO
- R10: value 100 -> 100k; LCSC Part No. C3508583 -> C513592; MPN (none) -> MF0207FTE52-100K; Manufacturer (none) -> YAGEO
- R11: value R_snub -> 10k; footprint Resistor_THT:R_Axial_DIN0411_L9.9mm_D3.6mm_P12.70mm_Horizontal -> Resistor_THT:R_Axial_DIN0207_L6.3mm_D2.5mm_P10.16mm_Horizontal; LCSC Part No. C385291 -> C513672; MPN (none) -> MF0207FTE52-10K; Manufacturer (none) -> YAGEO
- R12, R13: value 100 -> 1k; footprint Resistor_THT:R_Axial_DIN0207_L6.3mm_D2.5mm_P10.16mm_Horizontal -> Resistor_THT:R_Axial_DIN0411_L9.9mm_D3.6mm_P12.70mm_Horizontal; LCSC Part No. C3508583 -> C385291; MPN (none) -> RN1WS1KΩFT/BA1; Manufacturer (none) -> TyoHM; now not fitted; now left out of the parts list
- R16, R17: value 1k -> 100R; LCSC Part No. C513706 -> C3508583; MPN (none) -> MF0207FRE52-100R; Manufacturer (none) -> YAGEO
- R18: value R_snub -> 100R; footprint Resistor_THT:R_Axial_DIN0411_L9.9mm_D3.6mm_P12.70mm_Horizontal -> Resistor_THT:R_Axial_DIN0207_L6.3mm_D2.5mm_P10.16mm_Horizontal; LCSC Part No. C385291 -> C3508583; MPN (none) -> MF0207FRE52-100R; Manufacturer (none) -> YAGEO
- R19: value 33R -> 100R; LCSC Part No. (none) -> C3508583; MPN (none) -> MF0207FRE52-100R; Manufacturer (none) -> YAGEO
- R6: value 100k -> 100R; LCSC Part No. C513592 -> C3508583; MPN (none) -> MF0207FRE52-100R; Manufacturer (none) -> YAGEO
- R7: value 10k -> 100R; LCSC Part No. C513672 -> C3508583; MPN (none) -> MF0207FRE52-100R; Manufacturer (none) -> YAGEO
Connections:
- net +3V3 is gone; now on net +5V: U1.2 (VCC)
- net LowBattLED is gone; now on net A1: R17.1
- net +5V: now also A1.27 (+5V), C10.1, C11.1, C3.1, J4.5 (Pin_5), R9.1; no longer C1.1, R16.1, R6.1, U4.4 (Vs)
- net A1: now also J4.4 (Pin_4); no longer R12.1
- net A2: now also R18.1, J4.3 (Pin_3); no longer R13.1
- net GND: now also R11.2, A1.29 (GND), A1.4 (GND), C10.2, C11.2, C12.2, C2.2, C3.2, C4.2, D1.1 (K), D10.2 (A), D11.2 (A), D2.2 (A2), D6.2 (A), D7.2 (A), J1.1 (Pin_1), J4.1 (Pin_1); no longer R7.2
- net Radio_CE: now also R5.2; no longer R1.2
- net Radio_CS: now also R4.2; no longer R2.2
- net Radio_MISO: now also R2.2; no longer R4.2
- net Radio_SCK: now also R1.2; no longer R5.2
- net V_Panel_Analog: now also R10.2, R11.1, A1.25 (A6), C12.1; no longer R6.2, R7.1
- net at J3.1 (Pin_1): now also U4.2 (OUT1), C9.1, D4.2 (A), D6.1 (K); no longer U4.13 (OUT3)
- net at D3.2 (A): now also R14.2; no longer R16.2
- net at U4.3 (OUT2): now also J3.2 (Pin_2), R12.2, D5.2 (A), D7.1 (K); no longer R11.2
- net Radio_IRQ: now reaches U1.8 (IRQ)
- net Radio_IRQ: now also R6.2
- net A3: now reaches R19.1
- net A3: now also J4.2 (Pin_2)
- net at R19.2: now also A1.22 (A3)
- net at R1.1: now also A1.16 (D13)
- net at R4.1: now also A1.11 (D8)
- net at R17.2: now also A1.20 (A1)
- net at R2.1: now also A1.15 (D12)
- net at R3.1: now also A1.14 (D11)
- net at R5.1: now also A1.10 (D7)
- net at R13.2: now also U4.14 (OUT4), D11.1 (K), D9.2 (A), J2.2 (Pin_2)
- net A0 renamed PowerInput+
- net PowerInput+: now also C1.1, U4.4 (Vs), A1.30 (VIN), C2.1, C4.1, D2.1 (A1), D4.1 (K), D5.1 (K), D8.1 (K), D9.1 (K), F1.2
- net EnA renamed Motor_EnA
- net Motor_EnA: now also A1.12 (D9)
- net EnB renamed Motor_EnB
- net Motor_EnB: now also A1.13 (D10)
- net IN1 renamed Motor_IN1
- net Motor_IN1: now also R8.2
- net IN2 renamed Motor_IN2
- net Motor_IN2: now also R7.2
- net IN3 renamed Motor_IN3
- net Motor_IN3: now also R15.2
- net IN4 renamed Motor_IN4
- net Motor_IN4: now also R16.2
- new net: C8.2, R13.1
- new net: C9.2, R12.1
- new net: A1.21 (A2), R18.2
- new net: C8.1, D10.1 (K), D8.2 (A), J2.1 (Pin_1), U4.13 (OUT3)
- new net: F1.1, J1.2 (Pin_2)
- new net: D1.2 (A), R9.2
- new net: A1.7 (D4), R8.1
- new net: A1.8 (D5), R15.1
- new net: A1.5 (D2), R6.1
- new net: A1.9 (D6), R16.1
- new net: A1.6 (D3), R7.1
- new net LED1: A1.19 (A0), R14.1
- no-connect marks 11 -> 9
Other:
- note added: "do maths for this"
- note removed: "5V reg to step down and charge supercap as a backup power souce for any dip in power from input for Nano to use"
- note removed: "Extra Connector"
- note removed: "Power Backup"
- note removed: "for fun additions students want to add"
